Commit message: Added optional urdf transmissions to actuated joints, and added standalone gripper, for spot_choreo_utils web_animator

File: spot_description/urdf/spot.urdf.xacro (robot description, xacro)
@@ -25,4 +25,5 @@
   <xacro:arg name="k_q_p" default="" />
   <xacro:arg name="k_qd_p" default="" />
+  <xacro:arg name="include_transmissions" default="false" />
   <!-- Load Spot -->
   <xacro:load_spot
@@ -30,5 +31,6 @@
     feet="$(arg feet)"
     tf_prefix="$(arg tf_prefix)"
-    gripperless="$(arg gripperless)"/>
+		gripperless="$(arg gripperless)"
+		include_transmissions="$(arg include_transmissions)" />
   <!-- Adding the ROS 2 control tags -->
   <xacro:if value="$(arg add_ros2_control_tag)">

File: spot_description/urdf/spot_macro.xacro (robot description, xacro)
@@ -6,5 +6,6 @@
     gripperless:=false
     custom_gripper_base_link:=''
-    tf_prefix">
+			tf_prefix
+			include_transmissions=false">
         <link name="${tf_prefix}body">
             <visual>
@@ -81,4 +82,15 @@
                 upper="0.78539816339744827899" />
         </joint>
+        <xacro:if value="${include_transmissions}">
+					<transmission name="${tf_prefix}front_left_hip_x_tran">
+						<type>transmission_interface/SimpleTransmission</type>
+						<joint name="${tf_prefix}front_left_hip_x">
+							<hardwareInterface>EffortJointInterface</hardwareInterface>
+						</joint>
+						<actuator name="${tf_prefix}front_left_hip_x_motor">
+							<hardwareInterface>EffortJointInterface</hardwareInterface>
+						</actuator>
+					</transmission>
+        </xacro:if>
         <link name="${tf_prefix}front_left_upper_leg">
             <visual>
@@ -110,4 +122,15 @@
                 upper="2.2951079663725435509" />
         </joint>
+        <xacro:if value="${include_transmissions}">
+					<transmission name="${tf_prefix}front_left_hip_y_tran">
+						<type>transmission_interface/SimpleTransmission</type>
+						<joint name="${tf_prefix}front_left_hip_y">
+							<hardwareInterface>EffortJointInterface</hardwareInterface>
+						</joint>
+						<actuator name="${tf_prefix}front_left_hip_y_motor">
+							<hardwareInterface>EffortJointInterface</hardwareInterface>
+						</actuator>
+					</transmission>
+				</xacro:if>
         <link name="${tf_prefix}front_left_lower_leg">
             <visual>
@@ -137,4 +160,5 @@
             </inertial>
         </link>
+				<frame link="${tf_prefix}front_left_lower_leg" name="${tf_prefix}front_left_foot_center" xyz="0.0 0.0 -0.3365"/>
         <joint name="${tf_prefix}front_left_knee" type="revolute">
             <origin xyz="0.025 0.000 -0.3205" rpy="0 0 0" />
@@ -144,4 +168,15 @@
             <limit effort="115" velocity="12.0" lower="-2.7929" upper="-0.254801" />
         </joint>
+        <xacro:if value="${include_transmissions}">
+					<transmission name="${tf_prefix}front_left_knee_tran">
+						<type>transmission_interface/SimpleTransmission</type>
+						<joint name="${tf_prefix}front_left_knee">
+							<hardwareInterface>EffortJointInterface</hardwareInterface>
+						</joint>
+						<actuator name="${tf_prefix}front_left_knee_motor">
+							<hardwareInterface>EffortJointInterface</hardwareInterface>
+						</actuator>
+					</transmission>
+				</xacro:if>
         <link name="${tf_prefix}front_right_hip">
             <visual>
@@ -167,4 +202,15 @@
                 upper="0.78539816339744827899" />
         </joint>
+        <xacro:if value="${include_transmissions}">
+					<transmission name="${tf_prefix}front_right_hip_x_tran">
+						<type>transmission_interface/SimpleTransmission</type>
+						<joint name="${tf_prefix}front_right_hip_x">
+							<hardwareInterface>EffortJointInterface</hardwareInterface>
+						</joint>
+						<actuator name="${tf_prefix}front_right_hip_x_motor">
+							<hardwareInterface>EffortJointInterface</hardwareInterface>
+						</actuator>
+					</transmission>
+				</xacro:if>
         <link name="${tf_prefix}front_right_upper_leg">
             <visual>
@@ -196,4 +242,15 @@
                 upper="2.2951079663725435509" />
         </joint>
+        <xacro:if value="${include_transmissions}">
+					<transmission name="${tf_prefix}front_right_hip_y_tran">
+						<type>transmission_interface/SimpleTransmission</type>
+						<joint name="${tf_prefix}front_right_hip_y">
+							<hardwareInterface>EffortJointInterface</hardwareInterface>
+						</joint>
+						<actuator name="${tf_prefix}front_right_hip_y_motor">
+							<hardwareInterface>EffortJointInterface</hardwareInterface>
+						</actuator>
+					</transmission>
+				</xacro:if>
         <link name="${tf_prefix}front_right_lower_leg">
             <visual>
@@ -223,4 +280,5 @@
             </inertial>
         </link>
+				<frame link="${tf_prefix}front_right_lower_leg" name="${tf_prefix}front_right_foot_center" xyz="0.0 0.0 -0.3365"/>
         <joint name="${tf_prefix}front_right_knee" type="revolute">
             <origin xyz="0.025 0.000 -0.3205" rpy="0 0 0" />
@@ -230,4 +288,15 @@
             <limit effort="115" velocity="12.0" lower="-2.7929" upper="-0.247563" />
         </joint>
+        <xacro:if value="${include_transmissions}">
+					<transmission name="${tf_prefix}front_right_knee_tran">
+						<type>transmission_interface/SimpleTransmission</type>
+						<joint name="${tf_prefix}front_right_knee">
+							<hardwareInterface>EffortJointInterface</hardwareInterface>
+						</joint>
+						<actuator name="${tf_prefix}front_right_knee_motor">
+							<hardwareInterface>EffortJointInterface</hardwareInterface>
+						</actuator>
+					</transmission>
+				</xacro:if>
         <link name="${tf_prefix}rear_left_hip">
             <visual>
@@ -253,4 +322,15 @@
                 upper="0.78539816339744827899" />
         </joint>
+        <xacro:if value="${include_transmissions}">
+					<transmission name="${tf_prefix}rear_left_hip_x_tran">
+						<type>transmission_interface/SimpleTransmission</type>
+						<joint name="${tf_prefix}rear_left_hip_x">
+							<hardwareInterface>EffortJointInterface</hardwareInterface>
+						</joint>
+						<actuator name="${tf_prefix}rear_left_hip_x_motor">
+							<hardwareInterface>EffortJointInterface</hardwareInterface>
+						</actuator>
+					</transmission>
+				</xacro:if>
         <link name="${tf_prefix}rear_left_upper_leg">
             <visual>
@@ -282,4 +362,15 @@
                 upper="2.2951079663725435509" />
         </joint>
+        <xacro:if value="${include_transmissions}">
+					<transmission name="${tf_prefix}rear_left_hip_y_tran">
+						<type>transmission_interface/SimpleTransmission</type>
+						<joint name="${tf_prefix}rear_left_hip_y">
+							<hardwareInterface>EffortJointInterface</hardwareInterface>
+						</joint>
+						<actuator name="${tf_prefix}rear_left_hip_y_motor">
+							<hardwareInterface>EffortJointInterface</hardwareInterface>
+						</actuator>
+					</transmission>
+				</xacro:if>
         <link name="${tf_prefix}rear_left_lower_leg">
             <visual>
@@ -309,4 +400,5 @@
             </inertial>
         </link>
+				<frame link="${tf_prefix}rear_left_lower_leg" name="${tf_prefix}rear_left_foot_center" xyz="0.0 0.0 -0.3365"/>
         <joint name="${tf_prefix}rear_left_knee" type="revolute">
             <origin xyz="0.025 0.000 -0.3205" rpy="0 0 0" />
@@ -316,4 +408,15 @@
             <limit effort="115" velocity="12.0" lower="-2.7929" upper="-0.267153" />
         </joint>
+        <xacro:if value="${include_transmissions}">
+					<transmission name="${tf_prefix}rear_left_knee_tran">
+						<type>transmission_interface/SimpleTransmission</type>
+						<joint name="${tf_prefix}rear_left_knee">
+							<hardwareInterface>EffortJointInterface</hardwareInterface>
+						</joint>
+						<actuator name="${tf_prefix}rear_left_knee_motor">
+							<hardwareInterface>EffortJointInterface</hardwareInterface>
+						</actuator>
+					</transmission>
+				</xacro:if>
         <link name="${tf_prefix}rear_right_hip">
             <visual>
@@ -339,4 +442,15 @@
                 upper="0.78539816339744827899" />
         </joint>
+        <xacro:if value="${include_transmissions}">
+					<transmission name="${tf_prefix}rear_right_hip_x_tran">
+						<type>transmission_interface/SimpleTransmission</type>
+						<joint name="${tf_prefix}rear_right_hip_x">
+							<hardwareInterface>EffortJointInterface</hardwareInterface>
+						</joint>
+						<actuator name="${tf_prefix}rear_right_hip_x_motor">
+							<hardwareInterface>EffortJointInterface</hardwareInterface>
+						</actuator>
+					</transmission>
+				</xacro:if>
         <link name="${tf_prefix}rear_right_upper_leg">
             <visual>
@@ -368,4 +482,15 @@
                 upper="2.2951079663725435509" />
         </joint>
+        <xacro:if value="${include_transmissions}">
+					<transmission name="${tf_prefix}rear_right_hip_y_tran">
+						<type>transmission_interface/SimpleTransmission</type>
+						<joint name="${tf_prefix}rear_right_hip_y">
+							<hardwareInterface>EffortJointInterface</hardwareInterface>
+						</joint>
+						<actuator name="${tf_prefix}rear_right_hip_y_motor">
+							<hardwareInterface>EffortJointInterface</hardwareInterface>
+						</actuator>
+					</transmission>
+				</xacro:if>
         <link name="${tf_prefix}rear_right_lower_leg">
             <visual>
@@ -395,4 +520,5 @@
             </inertial>
         </link>
+				<frame link="${tf_prefix}rear_right_lower_leg" name="${tf_prefix}rear_right_foot_center" xyz="0.0 0.0 -0.3365"/>
         <joint name="${tf_prefix}rear_right_knee" type="revolute">
             <origin xyz="0.025 0.000 -0.3205" rpy="0 0 0" />
@@ -402,4 +528,15 @@
             <limit effort="115" velocity="12.0" lower="-2.7929" upper="-0.257725" />
         </joint>
+        <xacro:if value="${include_transmissions}">
+					<transmission name="${tf_prefix}rear_right_knee_tran">
+						<type>transmission_interface/SimpleTransmission</type>
+						<joint name="${tf_prefix}rear_right_knee">
+							<hardwareInterface>EffortJointInterface</hardwareInterface>
+						</joint>
+						<actuator name="${tf_prefix}rear_right_knee_motor">
+							<hardwareInterface>EffortJointInterface</hardwareInterface>
+						</actuator>
+					</transmission>
+        </xacro:if>
         <!-- Standard accessories. -->
         <xacro:include filename="$(find spot_description)/urdf/accessories.urdf.xacro" />

File: spot_description/urdf/standalone_arm.urdf.xacro (robot description, xacro)
@@ -6,6 +6,10 @@
   <!-- Parameters -->
   <xacro:arg name="tf_prefix" default="" />
+  <xacro:arg name="include_transmissions" default="false" />
+  <xacro:arg name="gripperless" default="false" />
   <!-- Load arm -->
   <xacro:load_arm
-    tf_prefix="$(arg tf_prefix)" />
+		tf_prefix="$(arg tf_prefix)"
+		gripperless="$(arg gripperless)"
+		include_transmissions="$(arg include_transmissions)"/>
 </robot>
